File: v2/kicad/spdif-decoder/spdif-decoder.kicad_pcb (KiCad board)
At the start: 2 copper layers, 73.7 x 80 mm, 30 parts, among them J1 DB25_Female, J2 TORX1350A_F_, SW1 SW_Push, U1 Teensy4.0, U2 74AHCT595, U3 74AHCT595, U4 74AHCT595, U5 74AHCT595

Commit message: mods, case
Parts:
- H1, H2, H3, H4: footprint MountingHole:MountingHole_4.3mm_M4 -> MountingHole:MountingHole_3.2mm_M3
- J2: value TORX1350A_F_ -> TORX1350A(F)
- moved H3 93.5 mm to (50.2, 145.4)
- moved H4 93.5 mm to (112.4, 145.4)
- moved H1 69.2 mm to (50.2, 76.8)
- moved H2 69.2 mm to (112.4, 76.8)
Other:
- outline, holes or cut-outs redrawn
- board text added: "0.1uF"
- board text added: "47uH"
- board text added: "560"
- board text added: "TORX1350A(F)"
