File: v2/kicad/spdif-decoder/spdif-decoder.sch (KiCad schematic (older format))
At the start: 30 parts, among them J1 DB25_Female, J2 TORX1350A_F_, SW1 SW_Push, U1 Teensy4.0, U2 74AHCT595, U3 74AHCT595, U4 74AHCT595, U5 74AHCT595

Commit message: mods, case
Parts:
- H1, H2, H3, H4: footprint MountingHole:MountingHole_4.3mm_M4 -> MountingHole:MountingHole_3.2mm_M3
Other:
- note added: "Configuration boot switch"
Changed lines of the file:
@@
 F 0 "H1" H 9200 1346 50  0000 L CNN
 F 1 "MountingHole" H 9200 1255 50  0000 L CNN
-F 2 "MountingHole:MountingHole_4.3mm_M4" H 9100 1300 50  0001 C CNN
+F 2 "MountingHole:MountingHole_3.2mm_M3" H 9100 1300 50  0001 C CNN
 F 3 "~" H 9100 1300 50  0001 C CNN
 	1    9100 1300
@@
 $Comp
 L Mechanical:MountingHole H2
-U 1 1 615A1A07
+U 1 1 615C6999
 P 9100 1500
 F 0 "H2" H 9200 1546 50  0000 L CNN
 F 1 "MountingHole" H 9200 1455 50  0000 L CNN
-F 2 "MountingHole:MountingHole_4.3mm_M4" H 9100 1500 50  0001 C CNN
+F 2 "MountingHole:MountingHole_3.2mm_M3" H 9100 1500 50  0001 C CNN
 F 3 "~" H 9100 1500 50  0001 C CNN
 	1    9100 1500
@@
 $Comp
 L Mechanical:MountingHole H3
-U 1 1 615A1D05
+U 1 1 615C6C1B
 P 9100 1700
 F 0 "H3" H 9200 1746 50  0000 L CNN
 F 1 "MountingHole" H 9200 1655 50  0000 L CNN
-F 2 "MountingHole:MountingHole_4.3mm_M4" H 9100 1700 50  0001 C CNN
+F 2 "MountingHole:MountingHole_3.2mm_M3" H 9100 1700 50  0001 C CNN
 F 3 "~" H 9100 1700 50  0001 C CNN
 	1    9100 1700
@@
 $Comp
 L Mechanical:MountingHole H4
-U 1 1 615A1F5C
+U 1 1 615C6ECB
 P 9100 1900
 F 0 "H4" H 9200 1946 50  0000 L CNN
 F 1 "MountingHole" H 9200 1855 50  0000 L CNN
-F 2 "MountingHole:MountingHole_4.3mm_M4" H 9100 1900 50  0001 C CNN
+F 2 "MountingHole:MountingHole_3.2mm_M3" H 9100 1900 50  0001 C CNN
 F 3 "~" H 9100 1900 50  0001 C CNN
 	1    9100 1900
 	1    0    0    -1
 $EndComp
+Text Notes 7050 750  0    50   ~ 0
+Configuration boot switch
 $EndSCHEMATC
